File: UART-RS485 Read only/UART-RS485 Read only.kicad_sch (KiCad schematic)
At the start: 21 parts, among them J1 Conn_01x02_Socket, J2 UART, J3 RS485, U1 MIC5504-3.3YM5, U2 MAX3485

Commit message: Add files via upload
Connections:
- net +5V: no longer J1.1 (Pin_1)
- net A: now also R6.1; no longer R5.1
- net B: now also R5.1; no longer R6.1
- net GND: no longer J1.2 (Pin_2)
- net at U2.2 (~{RE}), U2.3 (DE): now also J1.1 (Pin_1)
- no-connect marks 0 -> 1
Other:
- moved on the sheet: J1
Changed lines of the file:
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@@
 	)
 	(junction
+		(at 199.644 123.444)
+		(diameter 0)
+		(color 0 0 0 0)
+	)
+	(junction
 		(at 227.584 124.714)
 		(diameter 0)
@@
 		(color 0 0 0 0)
 	)
+	(no_connect
+		(at 183.388 111.506)
+	)
 	(wire
 		(pts
@@
 	(wire
 		(pts
-			(xy 77.216 44.704) (xy 80.264 44.704)
-		)
-		(stroke
-			(width 0)
-			(type default)
-		)
-	)
-	(wire
-		(pts
 			(xy 70.358 125.476) (xy 70.358 127.254)
 		)
@@
 	(wire
 		(pts
-			(xy 199.644 122.174) (xy 199.644 124.714)
+			(xy 199.644 123.444) (xy 199.644 124.714)
+		)
+		(stroke
+			(width 0)
+			(type default)
+		)
+	)
+	(wire
+		(pts
+			(xy 199.644 122.174) (xy 199.644 123.444)
 		)
 		(stroke
@@
 	(wire
 		(pts
+			(xy 180.848 111.506) (xy 180.848 123.444)
+		)
+		(stroke
+			(width 0)
+			(type default)
+		)
+	)
+	(wire
+		(pts
 			(xy 97.79 125.476) (xy 97.79 127.254)
 		)
@@
 	(wire
 		(pts
-			(xy 53.848 116.586) (xy 53.848 118.11)
+			(xy 180.848 123.444) (xy 199.644 123.444)
 		)
 		(stroke
@@
 	(wire
 		(pts
-			(xy 70.866 44.704) (xy 74.676 44.704)
+			(xy 53.848 116.586) (xy 53.848 118.11)
 		)
 		(stroke
@@
 	)
 	(label "A"
-		(at 89.154 108.712 180)
+		(at 97.79 108.712 180)
 		(fields_autoplaced yes)
 		(effects
@@
 	)
 	(label "B"
-		(at 97.79 108.712 180)
+		(at 89.154 108.712 180)
 		(fields_autoplaced yes)
 		(effects
@@
 	)
 	(symbol
-		(lib_id "power:+5V")
-		(at 70.866 44.704 0)
-		(unit 1)
-		(exclude_from_sim no)
-		(in_bom yes)
-		(on_board yes)
-		(dnp no)
-		(fields_autoplaced yes)
-		(property "Reference" "#PWR07"
-			(at 70.866 48.514 0)
-			(effects
-				(font
-					(size 1.27 1.27)
-				)
-				(hide yes)
-			)
-		)
-		(property "Value" "+5V"
-			(at 70.866 39.878 0)
-			(effects
-				(font
-					(size 1.27 1.27)
-				)
-			)
-		)
-		(property "Footprint" ""
-			(at 70.866 44.704 0)
-			(effects
-				(font
-					(size 1.27 1.27)
-				)
-				(hide yes)
-			)
-		)
-		(property "Datasheet" ""
-			(at 70.866 44.704 0)
-			(effects
-				(font
-					(size 1.27 1.27)
-				)
-				(hide yes)
-			)
-		)
-		(property "Description" "Power symbol creates a global label with name \"+5V\""
-			(at 70.866 44.704 0)
-			(effects
-				(font
-					(size 1.27 1.27)
-				)
-				(hide yes)
-			)
-		)
-		(pin "1"
-		)
-		(instances
-			(project "UART-RS485 Read only"
-				(path "/9bac4695-0bb8-42a3-8f69-7ad20dbe9ed8"
-					(reference "#PWR07")
-					(unit 1)
-				)
-			)
-		)
-	)
-	(symbol
 		(lib_id "power:+3.3V")
 		(at 209.804 109.474 0)
@@
 	)
 	(symbol
-		(lib_id "power:GND")
-		(at 80.264 44.704 0)
-		(unit 1)
-		(exclude_from_sim no)
-		(in_bom yes)
-		(on_board yes)
-		(dnp no)
-		(fields_autoplaced yes)
-		(property "Reference" "#PWR010"
-			(at 80.264 51.054 0)
-			(effects
-				(font
-					(size 1.27 1.27)
-				)
-				(hide yes)
-			)
-		)
-		(property "Value" "GND"
-			(at 80.264 49.276 0)
-			(effects
-				(font
-					(size 1.27 1.27)
-				)
-			)
-		)
-		(property "Footprint" ""
-			(at 80.264 44.704 0)
-			(effects
-				(font
-					(size 1.27 1.27)
-				)
-				(hide yes)
-			)
-		)
-		(property "Datasheet" ""
-			(at 80.264 44.704 0)
-			(effects
-				(font
-					(size 1.27 1.27)
-				)
-				(hide yes)
-			)
-		)
-		(property "Description" "Power symbol creates a global label with name \"GND\" , ground"
-			(at 80.264 44.704 0)
-			(effects
-				(font
-					(size 1.27 1.27)
-				)
-				(hide yes)
-			)
-		)
-		(pin "1"
-		)
-		(instances
-			(project "UART-RS485 Read only"
-				(path "/9bac4695-0bb8-42a3-8f69-7ad20dbe9ed8"
-					(reference "#PWR010")
-					(unit 1)
-				)
-			)
-		)
-	)
-	(symbol
 		(lib_id "Regulator_Linear:MIC5504-3.3YM5")
 		(at 104.14 52.07 0)
@@
 	(symbol
 		(lib_id "Connector:Conn_01x02_Socket")
-		(at 74.676 39.624 90)
+		(at 180.848 106.426 90)
 		(unit 1)
 		(exclude_from_sim no)
@@
 		(dnp no)
 		(property "Reference" "J1"
-			(at 74.676 34.036 90)
+			(at 180.848 100.838 90)
 			(effects
 				(font
@@
 		)
 		(property "Value" "Conn_01x02_Socket"
-			(at 67.056 36.322 90)
+			(at 173.228 103.124 90)
 			(effects
 				(font
@@
 		)
 		(property "Footprint" "Connector_JST:JST_XA_S02B-XASK-1_1x02_P2.50mm_Horizontal"
-			(at 74.676 39.624 0)
+			(at 180.848 106.426 0)
 			(effects
 				(font
@@
 		)
 		(property "Datasheet" "~"
-			(at 74.676 39.624 0)
+			(at 180.848 106.426 0)
 			(effects
 				(font
@@
 		)
 		(property "Description" "Generic connector, single row, 01x02, script generated"
-			(at 74.676 39.624 0)
+			(at 180.848 106.426 0)
 			(effects
 				(font
